File: Kicad/x399 REF.kicad_pcb (KiCad board)
At the start: 2 copper layers, 106 x 56 mm, 57 parts, among them J1 +15V, J2 10Vref, Q1 MMBT3904, Q2 2SD882, U1 LM399, U2 OP07

Commit message: Add files via upload
Parts:
- D1, D4, D5: value STPS130 -> SS34A
- R9: value 220k -> Calc

Commit message: Board revision
Rotated LM399 to have sensitive to TEMF pins (1,2) perpendicular to thermal gradient
Parts:
- moved C1 28.8 mm to (93.2, 99.4), turned to 180 degrees
- moved C2 22.7 mm to (131.6, 105.4), turned to 90 degrees
- moved R2 20.9 mm to (131.5, 110.0), turned to -90 degrees
- moved U1 3.03 mm to (113.5, 110.9), turned to 180 degrees
Routing:
- net Net-(U2A-+): track 101.8 -> 150.3 mm, vias 11 -> 8
- net MGND: track 147.2 -> 183.1 mm, vias 8 -> 12
- net Earth: track 172.3 -> 157.4 mm, vias 475 -> 341
- net +10VREF: track 198.8 -> 196.6 mm

Commit message: Board revision
Rotate transistor so it can be mounted to enclosure for heatsinking
Parts:
- moved Q2 8.28 mm to (77.5, 70.2), turned to 0 degrees
- moved R13 6.04 mm to (77.6, 76.9)
- moved D3 4.60 mm to (85.4, 71.0), turned to -90 degrees
- moved C10 4.54 mm to (71.7, 79.5)
- moved Q1 3.90 mm to (74.6, 80.1)
- moved D4 2.91 mm to (80.8, 77.7)
- moved R10 0.25 mm to (85.1, 74.9)
Routing:
- net MGND: track 183.1 -> 207.5 mm
- net Earth: track 157.4 -> 172.2 mm, vias 341 -> 346
- net Net-(D4-K): track 50.3 -> 60.4 mm
- net +10VREF: track 196.6 -> 204.6 mm
- net Net-(D3-K): track 52.2 -> 48.0 mm, vias 2 -> 0
- net Net-(U2A-+): track 150.3 -> 151.3 mm
- net Net-(Q1-B): track 22.2 -> 22.3 mm, vias 0 -> 4
Other:
- outline, holes or cut-outs redrawn

Commit message: Add files via upload
Routing:
- net MGND: track 207.5 -> 282.2 mm, vias 12 -> 13
- net +10VREF: track 204.6 -> 203.8 mm
- net Earth: vias 346 -> 342
